File: TurboXT.sch (KiCad schematic (older format))
At the start: 25 parts, among them J1 8284 Socket, J2 HRQDMA, J3 DMAWAIT, J4 VCC, J5 GND, J6 Turbo LED, SW1 TURBO SWITCH, U1 8284, U2 74LS92, U3 74LS74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

Commit message: Updated silkscreen
Parts:
- U7: value 74LS14 -> 74HCT14
Changed lines of the file:
@@
 Title "TurboXT"
 Date ""
-Rev "1.1"
+Rev "1.2"
 Comp ""
 Comment1 "Copyright (c) 2014 Sergey Kiselev"
@@
 P 2950 2000
 F 0 "U7" H 2950 2317 50  0000 C CNN
-F 1 "74LS14" H 2950 2226 50  0000 C CNN
+F 1 "74HCT14" H 2950 2226 50  0000 C CNN
 F 2 "Package_DIP:DIP-14_W7.62mm_LongPads" H 2950 2000 50  0001 C CNN
 F 3 "http://www.ti.com/lit/gpn/sn74LS14" H 2950 2000 50  0001 C CNN
@@
 P 9700 5600
 F 0 "U7" H 9930 5646 50  0000 L CNN
-F 1 "74LS14" H 9930 5555 50  0000 L CNN
+F 1 "74HCT14" H 9930 5555 50  0000 L CNN
 F 2 "Package_DIP:DIP-14_W7.62mm_LongPads" H 9700 5600 50  0001 C CNN
 F 3 "http://www.ti.com/lit/gpn/sn74LS14" H 9700 5600 50  0001 C CNN
@@
 P 2950 2500
 F 0 "U7" H 2950 2817 50  0000 C CNN
-F 1 "74LS14" H 2950 2726 50  0000 C CNN
+F 1 "74HCT14" H 2950 2726 50  0000 C CNN
 F 2 "Package_DIP:DIP-14_W7.62mm_LongPads" H 2950 2500 50  0001 C CNN
 F 3 "http://www.ti.com/lit/gpn/sn74LS14" H 2950 2500 50  0001 C CNN
@@
 P 5600 3300
 F 0 "U7" H 5600 3617 50  0000 C CNN
-F 1 "74LS14" H 5600 3526 50  0000 C CNN
+F 1 "74HCT14" H 5600 3526 50  0000 C CNN
 F 2 "Package_DIP:DIP-14_W7.62mm_LongPads" H 5600 3300 50  0001 C CNN
 F 3 "http://www.ti.com/lit/gpn/sn74LS14" H 5600 3300 50  0001 C CNN
@@
 P 5600 3800
 F 0 "U7" H 5600 4117 50  0000 C CNN
-F 1 "74LS14" H 5600 4026 50  0000 C CNN
+F 1 "74HCT14" H 5600 4026 50  0000 C CNN
 F 2 "Package_DIP:DIP-14_W7.62mm_LongPads" H 5600 3800 50  0001 C CNN
 F 3 "http://www.ti.com/lit/gpn/sn74LS14" H 5600 3800 50  0001 C CNN
@@
 P 5600 4300
 F 0 "U7" H 5600 4617 50  0000 C CNN
-F 1 "74LS14" H 5600 4526 50  0000 C CNN
+F 1 "74HCT14" H 5600 4526 50  0000 C CNN
 F 2 "Package_DIP:DIP-14_W7.62mm_LongPads" H 5600 4300 50  0001 C CNN
 F 3 "http://www.ti.com/lit/gpn/sn74LS14" H 5600 4300 50  0001 C CNN
@@
 P 5600 4800
 F 0 "U7" H 5600 5117 50  0000 C CNN
-F 1 "74LS14" H 5600 5026 50  0000 C CNN
+F 1 "74HCT14" H 5600 5026 50  0000 C CNN
 F 2 "Package_DIP:DIP-14_W7.62mm_LongPads" H 5600 4800 50  0001 C CNN
 F 3 "http://www.ti.com/lit/gpn/sn74LS14" H 5600 4800 50  0001 C CNN

Commit message: Add reset button
Parts:
- added J7: Reset, Connector_PinHeader_2.54mm:PinHeader_1x02_P2.54mm_Vertical, symbol Connector_Generic:Conn_01x02
- added R4: 10k, Resistor_THT:R_Axial_DIN0207_L6.3mm_D2.5mm_P10.16mm_Horizontal, symbol Device:R_Small
Connections:
- net GND: now also J7.1 (Pin_1)
- net ~RES: now also J7.2 (Pin_2), R4.2; no longer J1.11 (Pin_11)
- new net: J1.11 (Pin_11), R4.1
Changed lines of the file:
@@
 Wire Wire Line
 	5750 6200 6200 6200
-Wire Wire Line
-	5750 6300 6200 6300
-Wire Wire Line
-	5750 6400 6200 6400
 Text Label 4850 5600 0    50   ~ 0
 CSYNC
@@
 Text Label 6200 6400 2    50   ~ 0
 RESET
-Text Label 6200 6300 2    50   ~ 0
+Text Label 6500 6300 2    50   ~ 0
 ~RES
 Text Label 6200 6200 2    50   ~ 0
@@
 Text Label 2500 4200 0    50   ~ 0
 RESET
+$Comp
+L Device:R_Small R4
+U 1 1 60B40AA8
+P 6100 6300
+F 0 "R4" V 6150 6400 50  0000 L CNN
+F 1 "10k" V 6150 6050 50  0000 L CNN
+F 2 "Resistor_THT:R_Axial_DIN0207_L6.3mm_D2.5mm_P10.16mm_Horizontal" H 6100 6300 50  0001 C CNN
+F 3 "~" H 6100 6300 50  0001 C CNN
+	1    6100 6300
+	0    -1   -1   0
+$EndComp
+$Comp
+L Connector_Generic:Conn_01x02 J7
+U 1 1 60B71C6D
+P 6150 6600
+F 0 "J7" H 6230 6592 50  0000 L CNN
+F 1 "Reset" H 6230 6501 50  0000 L CNN
+F 2 "Connector_PinHeader_2.54mm:PinHeader_1x02_P2.54mm_Vertical" H 6150 6600 50  0001 C CNN
+F 3 "~" H 6150 6600 50  0001 C CNN
+	1    6150 6600
+	-1   0    0    1
+$EndComp
+Wire Wire Line
+	6350 6500 6500 6500
+Wire Wire Line
+	6500 6500 6500 6300
+$Comp
+L power:GND #PWR?
+U 1 1 60B7B2DF
+P 6500 6700
+F 0 "#PWR?" H 6500 6450 50  0001 C CNN
+F 1 "GND" H 6505 6527 50  0000 C CNN
+F 2 "" H 6500 6700 50  0001 C CNN
+F 3 "" H 6500 6700 50  0001 C CNN
+	1    6500 6700
+	1    0    0    -1
+$EndComp
+Wire Wire Line
+	5750 6400 6200 6400
+Wire Wire Line
+	6000 6300 5750 6300
+Wire Wire Line
+	6200 6300 6500 6300
+Wire Wire Line
+	6350 6600 6500 6600
+Wire Wire Line
+	6500 6600 6500 6700
 $EndSCHEMATC

Commit message: Add cap for deboucing
Parts:
- added C9: 100nF, Capacitor_THT:C_Disc_D6.0mm_W2.5mm_P5.00mm, symbol Device:C_Small
Connections:
- net GND: now also C9.2
- net ~RES: now also C9.1
Changed lines of the file:
@@
 	6350 6500 6500 6500
 Wire Wire Line
-	6500 6500 6500 6300
+	6500 6500 6500 6450
 $Comp
 L power:GND #PWR?
@@
 	6350 6600 6500 6600
 Wire Wire Line
-	6500 6600 6500 6700
+	6500 6600 6500 6650
+$Comp
+L Device:C_Small C9
+U 1 1 60B18C33
+P 6600 6550
+F 0 "C9" H 6692 6596 50  0000 L CNN
+F 1 "100nF" H 6692 6505 50  0000 L CNN
+F 2 "Capacitor_THT:C_Disc_D6.0mm_W2.5mm_P5.00mm" H 6600 6550 50  0001 C CNN
+F 3 "~" H 6600 6550 50  0001 C CNN
+	1    6600 6550
+	1    0    0    -1
+$EndComp
+Wire Wire Line
+	6600 6650 6500 6650
+Connection ~ 6500 6650
+Wire Wire Line
+	6500 6650 6500 6700
+Wire Wire Line
+	6600 6450 6500 6450
+Connection ~ 6500 6450
+Wire Wire Line
+	6500 6450 6500 6300
 $EndSCHEMATC
